Commit message: add mujoco sim

File: robot_description/tita_description/xacro/description.xacro (robot description, xacro)
@@ -53,5 +53,5 @@
     </visual>
     <collision>
-      <origin
+      <!-- <origin
         xyz="0 0 0"
         rpy="0 0 0" />
@@ -59,4 +59,10 @@
         <mesh
           filename="package://tita_description/meshes/base_link.STL" />
+      </geometry> -->
+      <origin
+        rpy="0 0 0"
+        xyz="0 0 0.017"/>
+      <geometry>
+        <box size="0.47 0.3 0.19"/>
       </geometry>
     </collision>
@@ -121,5 +127,5 @@
       </material>
     </visual>
-    <collision>
+    <!-- <collision>
       <origin
         xyz="0 0 0"
@@ -129,5 +135,5 @@
           filename="package://tita_description/meshes/left_hip.STL" />
       </geometry>
-    </collision>
+    </collision> -->
   </link>
   <joint
@@ -144,8 +150,8 @@
       xyz="0 0 1" />
     <limit
-      lower="-0.4"
-      upper="0.4"
-      effort="53"
-      velocity="18.84" />
+      lower="-0.785398"
+      upper="0.785398"
+      effort="60"
+      velocity="25" />
   </joint>
   <link
@@ -180,5 +186,5 @@
     </visual>
     <collision>
-      <origin
+      <!-- <origin
         xyz="0 0 0"
         rpy="0 0 0" />
@@ -186,4 +192,10 @@
         <mesh
           filename="package://tita_description/meshes/left_thigh.STL" />
+      </geometry> -->
+      <origin
+        rpy="0 0 -0.131"
+        xyz="0.1 0.021 -0.002"/>
+      <geometry>
+        <box size="0.2 0.09 0.05"/>
       </geometry>
     </collision>
@@ -202,8 +214,8 @@
       xyz="0 0 1" />
     <limit
-      lower="-1.5708"
-      upper="1.5708"
-      effort="53"
-      velocity="18.84" />
+      lower="-1.919862"
+      upper="3.490659"
+      effort="60"
+      velocity="25" />
   </joint>
   <link
@@ -238,5 +250,5 @@
     </visual>
     <collision>
-      <origin
+      <!-- <origin
         xyz="0 0 0"
         rpy="0 0 0" />
@@ -244,4 +256,10 @@
         <mesh
           filename="package://tita_description/meshes/left_calf.STL" />
+      </geometry> -->
+      <origin
+        rpy="0 0 -0.131"
+        xyz="0.1 0.021 -0.002"/>
+      <geometry>
+        <box size="0.2 0.07 0.05"/>
       </geometry>
     </collision>
@@ -260,8 +278,8 @@
       xyz="0 0 1" />
     <limit
-      lower="-2.672"
-      upper="-0.83776"
-      effort="53"
-      velocity="18.84" />
+      lower="-2.670354"
+      upper="-0.698132"
+      effort="60"
+      velocity="25" />
   </joint>
   <link
@@ -296,5 +314,5 @@
     </visual>
     <collision>
-      <origin
+      <!-- <origin
         xyz="0 0 0"
         rpy="0 0 0" />
@@ -302,4 +320,10 @@
         <mesh
           filename="package://tita_description/meshes/left_wheel.STL" />
+      </geometry> -->
+      <origin
+        rpy="0 0 0"
+        xyz="0 0 0"/>
+      <geometry>
+        <cylinder length="0.034" radius="0.0925"/>
       </geometry>
     </collision>
@@ -320,6 +344,6 @@
          lower=" -10000000000000.0"
       upper="10000000000000.0"
-      effort="10"
-      velocity="104.88" />
+      effort="15"
+      velocity="20" />
   </joint>
   <link
@@ -353,5 +377,5 @@
       </material>
     </visual>
-    <collision>
+    <!-- <collision>
       <origin
         xyz="0 0 0"
@@ -361,5 +385,5 @@
           filename="package://tita_description/meshes/right_hip.STL" />
       </geometry>
-    </collision>
+    </collision> -->
   </link>
   <joint
@@ -376,8 +400,8 @@
       xyz="0 0 1" />
     <limit
-      lower="-0.4"
-      upper="0.4"
-      effort="53"
-      velocity="18.84" />
+      lower="-0.785398"
+      upper="0.785398"
+      effort="60"
+      velocity="25" />
   </joint>
   <link
@@ -412,5 +436,5 @@
     </visual>
     <collision>
-      <origin
+      <!-- <origin
         xyz="0 0 0"
         rpy="0 0 0" />
@@ -418,4 +442,10 @@
         <mesh
           filename="package://tita_description/meshes/right_thigh.STL" />
+      </geometry> -->
+      <origin
+        rpy="0 0 -0.131"
+        xyz="0.1 0.021 -0.002"/>
+      <geometry>
+        <box size="0.2 0.09 0.05"/>
       </geometry>
     </collision>
@@ -432,10 +462,10 @@
       link="right_thigh" />
     <axis
-      xyz="0 0 -1" />
-    <limit
-      lower="-1.5708"
-      upper="1.5708"
-      effort="53"
-      velocity="18.84" />
+      xyz="0 0 1" />
+    <limit
+      lower="-1.919862"
+      upper="3.490659"
+      effort="60"
+      velocity="25" />
   </joint>
   <link
@@ -470,5 +500,5 @@
     </visual>
     <collision>
-      <origin
+      <!-- <origin
         xyz="0 0 0"
         rpy="0 0 0" />
@@ -476,4 +506,10 @@
         <mesh
           filename="package://tita_description/meshes/right_calf.STL" />
+      </geometry> -->
+      <origin
+        rpy="0 0 -0.131"
+        xyz="0.1 0.021 -0.002"/>
+      <geometry>
+        <box size="0.2 0.07 0.05"/>
       </geometry>
     </collision>
@@ -490,10 +526,10 @@
       link="right_calf" />
     <axis
-      xyz="0 0 -1" />
-    <limit
-      lower="0.83776"
-      upper="2.672"
-      effort="53"
-      velocity="18.84" />
+      xyz="0 0 1" />
+    <limit
+      lower="-2.670354"
+      upper="-0.698132"
+      effort="60"
+      velocity="25" />
   </joint>
   <link
@@ -528,5 +564,5 @@
     </visual>
     <collision>
-      <origin
+      <!-- <origin
         xyz="0 0 0"
         rpy="0 0 0" />
@@ -534,4 +570,10 @@
         <mesh
           filename="package://tita_description/meshes/right_wheel.STL" />
+      </geometry> -->
+      <origin
+        rpy="0 0 0"
+        xyz="0 0 0"/>
+      <geometry>
+        <cylinder length="0.034" radius="0.0925"/>
       </geometry>
     </collision>
@@ -548,10 +590,10 @@
       link="right_wheel" />
     <axis
-      xyz="0 0 -1" />
+      xyz="0 0 1" />
     <limit
      lower=" -10000000000000.0"
       upper="10000000000000.0"
-      effort="10"
-      velocity="104.88" />
+      effort="15"
+      velocity="20" />
   </joint>
     </xacro:macro>

File: robot_description/tita_description/xacro/ros2_control.xacro (robot description, xacro)
@@ -15,6 +15,6 @@
                 <command_interface name="velocity"/>
                 <command_interface name="effort">
-                    <param name="min">-53</param>
-                    <param name="max">53</param>
+                    <param name="min">-60</param>
+                    <param name="max">60</param>
                 </command_interface>
                 <command_interface name="kp"/>
@@ -30,11 +30,11 @@
                 <command_interface name="velocity"/>
                 <command_interface name="effort">
-                    <param name="min">-53</param>
-                    <param name="max">53</param>
-                </command_interface>
-                <command_interface name="kp"/>
-                <command_interface name="kd"/>
-                <state_interface name="position">
-                    <param name="initial_value">1.3</param>
+                    <param name="min">-60</param>
+                    <param name="max">60</param>
+                </command_interface>
+                <command_interface name="kp"/>
+                <command_interface name="kd"/>
+                <state_interface name="position">
+                    <param name="initial_value">0.8</param>
                 </state_interface>
                 <state_interface name="velocity"/>
@@ -45,11 +45,11 @@
                 <command_interface name="velocity"/>
                 <command_interface name="effort">
-                    <param name="min">-53</param>
-                    <param name="max">53</param>
-                </command_interface>
-                <command_interface name="kp"/>
-                <command_interface name="kd"/>
-                <state_interface name="position">
-                    <param name="initial_value">-2.6</param>
+                    <param name="min">-60</param>
+                    <param name="max">60</param>
+                </command_interface>
+                <command_interface name="kp"/>
+                <command_interface name="kd"/>
+                <state_interface name="position">
+                    <param name="initial_value">-1.5</param>
                 </state_interface>
                 <state_interface name="velocity"/>
@@ -60,6 +60,6 @@
                 <command_interface name="velocity"/>
                 <command_interface name="effort">
-                    <param name="min">-10</param>
-                    <param name="max">10</param>
+                    <param name="min">-15</param>
+                    <param name="max">15</param>
                 </command_interface>
                 <command_interface name="kp"/>
@@ -75,6 +75,6 @@
                 <command_interface name="velocity"/>
                 <command_interface name="effort">
-                    <param name="min">-53</param>
-                    <param name="max">53</param>
+                    <param name="min">-60</param>
+                    <param name="max">60</param>
                 </command_interface>
                 <command_interface name="kp"/>
@@ -90,11 +90,11 @@
                 <command_interface name="velocity"/>
                 <command_interface name="effort">
-                    <param name="min">-53</param>
-                    <param name="max">53</param>
-                </command_interface>
-                <command_interface name="kp"/>
-                <command_interface name="kd"/>
-                <state_interface name="position">
-                    <param name="initial_value">-1.3</param>
+                    <param name="min">-60</param>
+                    <param name="max">60</param>
+                </command_interface>
+                <command_interface name="kp"/>
+                <command_interface name="kd"/>
+                <state_interface name="position">
+                    <param name="initial_value">0.8</param>
                 </state_interface>
                 <state_interface name="velocity"/>
@@ -105,11 +105,11 @@
                 <command_interface name="velocity"/>
                 <command_interface name="effort">
-                    <param name="min">-53</param>
-                    <param name="max">53</param>
-                </command_interface>
-                <command_interface name="kp"/>
-                <command_interface name="kd"/>
-                <state_interface name="position">
-                    <param name="initial_value">2.6</param>
+                    <param name="min">-60</param>
+                    <param name="max">60</param>
+                </command_interface>
+                <command_interface name="kp"/>
+                <command_interface name="kd"/>
+                <state_interface name="position">
+                    <param name="initial_value">-1.5</param>
                 </state_interface>
                 <state_interface name="velocity"/>
@@ -120,6 +120,6 @@
                 <command_interface name="velocity"/>
                 <command_interface name="effort">
-                    <param name="min">-10</param>
-                    <param name="max">10</param>
+                    <param name="min">-15</param>
+                    <param name="max">15</param>
                 </command_interface>
                 <command_interface name="kp"/>
@@ -160,5 +160,5 @@
                 <sensor name="imu" type="imu">
                     <always_on>true</always_on>
-                    <update_rate>500</update_rate>
+                    <update_rate>1000</update_rate>
                 </sensor>
             </gazebo>
@@ -167,5 +167,5 @@
             </gazebo>
             <gazebo reference="base_link">
-                <self_collide>false</self_collide>
+                <self_collide>true</self_collide>
                 <gravity>true</gravity>
                 <mu1>1.0</mu1>
@@ -179,5 +179,5 @@
             </gazebo>
             <gazebo reference="joint_left_hip">
-                <self_collide>false</self_collide>
+                <self_collide>true</self_collide>
                 <gravity>true</gravity>
                 <mu1>1.0</mu1>
@@ -185,5 +185,5 @@
             </gazebo>
             <gazebo reference="joint_left_thigh">
-                <self_collide>false</self_collide>
+                <self_collide>true</self_collide>
                 <gravity>true</gravity>
                 <mu1>1.0</mu1>
@@ -193,5 +193,5 @@
             </gazebo>
             <gazebo reference="joint_left_calf">
-                <self_collide>false</self_collide>
+                <self_collide>true</self_collide>
                 <gravity>true</gravity>
                 <mu1>1.0</mu1>
@@ -201,13 +201,13 @@
             </gazebo>
             <gazebo reference="joint_left_wheel">
-                <self_collide>false</self_collide>
-                <gravity>true</gravity>
-                <mu1>1.0</mu1>
-                <mu2>1.0</mu2>
+                <self_collide>true</self_collide>
+                <gravity>true</gravity>
+                <mu1>2.0</mu1>
+                <mu2>2.0</mu2>
                 <kp  value="1000000.0"/>
                 <kd  value="1.0"/>
             </gazebo>
             <gazebo reference="joint_right_hip">
-                <self_collide>false</self_collide>
+                <self_collide>true</self_collide>
                 <gravity>true</gravity>
                 <mu1>1.0</mu1>
@@ -215,5 +215,5 @@
             </gazebo>
             <gazebo reference="joint_right_thigh">
-                <self_collide>false</self_collide>
+                <self_collide>true</self_collide>
                 <gravity>true</gravity>
                 <mu1>1.0</mu1>
@@ -223,5 +223,5 @@
             </gazebo>
             <gazebo reference="joint_right_calf">
-                <self_collide>false</self_collide>
+                <self_collide>true</self_collide>
                 <gravity>true</gravity>
                 <mu1>1.0</mu1>
@@ -231,8 +231,8 @@
             </gazebo>
             <gazebo reference="joint_right_wheel">
-                <self_collide>false</self_collide>
-                <gravity>true</gravity>
-                <mu1>1.0</mu1>
-                <mu2>1.0</mu2>
+                <self_collide>true</self_collide>
+                <gravity>true</gravity>
+                <mu1>2.0</mu1>
+                <mu2>2.0</mu2>
                 <kp  value="1000000.0"/>
                 <kd  value="1.0"/>
@@ -240,5 +240,5 @@
             <gazebo>
                 <is_static>true</is_static>
-                <self_collide>false</self_collide>
+                <self_collide>true</self_collide>
             </gazebo>
         </xacro:if>
